Commit message: fix: apt版driver(v0.2.2)のoffset方式へ全面的に書き直す
■ 根本原因
実機の /joint_states が Present * 2pi/4096 と完全一致していた
(elbow_flex: 1847 * 2pi/4096 = 2.8333 = 報告値)。2048 を引いておらず
全関節が +pi rad ずれていた。

原因は、私が GitHub main のソースを読んで設計していたのに、実機には
apt の v0.2.2 が入っていたこと。両者はパラメータの意味が全く違う。

  機能                v0.2.2 (実機)          main (私が読んでいた)
  中心値              per-joint の offset    kStsMidpoint(2048) 固定
  offset              必須。無いと 0         非推奨・無視
  PID の綴り          p_cofficient (e抜け)   p_coefficient
  joint_config_file   無い                   ある
  homing_offset       無い                   ある (EEPROMへ書く)
  range_min/max       無い                   ある (EEPROMへ書く)

私が「上流のバグ」として直した3点は、すべて v0.2.2 では正しい記述だった。
- offset を削除 -> これが今回の原因
- p_cofficient を「正しい綴り」に修正 -> PID が一度も効いていなかった
- joint_config_file を追加 -> v0.2.2 に無く so101_joints.yaml は完全に無視されていた

副次的に判明: homing_offset/range_* は v0.2.2 に無いので、サーボの EEPROM は
**一度も書き換わっていない**。較正値は lerobot が書いたまま無傷。

■ 修正
- control/so101_follower.ros2_control.xacro を offset 方式へ全面書き換え。
  PID は v0.2.2 に合わせて意図的に p_cofficient と綴る
- config/so101_offsets.xacro を新設し、機体の offset を分離
  (2052 / 1978 / 1916 / 2182 / 2048 / 1961)
- so101_calib に emit_xacro を追加し、可動域から offset を生成できるようにした
- Dockerfile に driver のバージョン検査を追加。0.2.2 以外ならビルドを止める
- スモークテストを v0.2.2 前提へ更新 (offset と p_cofficient の存在を確認し、
  joint_config_file が無いことを確認。offset 6個が 0..4095 に収まることも検査)
- setup.py が config/*.xacro を install するよう修正

■ 注意点
XML コメント内に連続ハイフンを書けない。--rm や --from-servos を含む
コマンド例を貼ってパースに失敗した。コマンド例は README 側に置くこと。

EEPROM を書き換えないので、この方式は較正値を壊す心配が無い。

Co-Authored-By: Claude <noreply@anthropic.com>

File: ros2_ws/src/so101_bringup/control/so101_follower.ros2_control.xacro (robot description, xacro)
@@ -2,29 +2,31 @@
 <!--
   SO-101 follower 用の ros2_control 記述。
-  ■ なぜ上流のファイルを使わないのか
-  上流 (ros-physical-ai/ros2_so_arm) の
-  so_arm101_description/control/so_arm101.ros2_control.xacro には、
-  feetech_ros2_driver v0.2.2 のソースと突き合わせて確認した実バグが3つある:
-    1. <param name="offset">2048</param> を設定しているが、driver 側で offset は
-       **非推奨で無視される**。起動時に警告が6回出るだけで何も反映されない。
-    2. PID パラメータの綴りが "p_cofficient" (e が抜けている)。driver は
-       "p_coefficient" を探すので、**PID 値は一切書き込まれない**。
-    3. joint_config_file のハードウェアパラメータが無いため、
-       **較正 YAML を渡す口が無い**。
-  幸い上流の親 xacro (so_arm101.urdf.xacro) には ros2_control_file:= という
-  差し替え用の引数があるので、URDF 本体はフォークせずこのファイルだけを渡す。
-  マクロ名と引数 (prefix ros2_control_hardware_type usb_port) は上流と同一に保つこと。
-  ■ 設計方針
-  関節ごとに書くのは **id だけ**。PID・加速度・保護電流・較正値はすべて
-  config/so101_joints.yaml 側に置く。driver は YAML を **joint 名ではなく id**
-  で突合せ、YAML が URDF より優先される。設定が二箇所に散らないようにする。
-  mujoco / gazebo の分岐は落としてある (スコープ外。かつ mujoco 分岐は
-  MuJoCo ランタイムを同梱していないのに mjcf/scene.xml を参照してしまう)。
+  ★★★ 対象は apt の feetech_ros2_driver **v0.2.2**。GitHub の main とは別物。★★★
+  ■ v0.2.2 と main の違い（実機で判明。ここを取り違えると全関節が π rad ずれる）
+  機能                  apt v0.2.2                    GitHub main
+  ....................  ............................  ............................
+  中心値の扱い          per-joint の `offset`         `kStsMidpoint`(2048) 固定
+  `offset`              必須。無いと 0 になる         非推奨・無視される
+  PID の綴り            `p_cofficient`（e 抜け）      `p_coefficient`
+  `joint_config_file`   無い                          ある
+  `homing_offset`       無い                          ある（EEPROM へ書く）
+  `range_min/max`       無い                          ある（EEPROM へ書く）
+  v0.2.2 の read/write は
+      read : q   = to_radians(Present - offset)
+      write: tick = from_radians(q) + offset
+  なので **`offset` = URDF ゼロ姿勢における Present の tick 値**。
+  `offset` を書かないと 0 になり、`q = Present * 2π/4096` すなわち
+  全関節が **+π rad** ずれる。RViz が不可能な姿勢になり、
+  `joint_limiter_interface` が limit 超過で例外を投げてコントローラが落ちる。
+  ■ v0.2.2 では EEPROM を書き換えない
+  `offset` は純粋なソフト側の値で、サーボの EEPROM には触らない。
+  較正値（homing_offset / range）は lerobot が書いたものがそのまま残り、
+  この構成からは変更されない。**壊す心配が無いのは利点。**
+  ■ offset の値
+  `config/so101_offsets.xacro` に分離してある。機体ごとの較正値なのでそちら参照。
 -->
 <robot xmlns:xacro="http://www.ros.org/wiki/xacro">
-  <xacro:arg
-    name="joint_config_file"
-    default="$(find so101_bringup)/config/so101_joints.yaml"
-  />
+  <!-- 機体ごとの offset（URDF ゼロにおける Present tick）-->
+  <xacro:include filename="$(find so101_bringup)/config/so101_offsets.xacro"/>
   <xacro:macro
     name="ros2_control"
@@ -40,49 +42,29 @@
           <plugin>feetech_ros2_driver/FeetechHardwareInterface</plugin>
           <param name="usb_port">${usb_port}</param>
-          <!-- ★ 上流に無い。較正値と調整値はすべてこの YAML から入る。 -->
-          <param name="joint_config_file">$(arg joint_config_file)</param>
         </xacro:if>
       </hardware>
       <!--
-        関節の並びは URDF (so_arm101_macro.xacro) と、
-        config/ros2_controllers.yaml の joints リストに一致させること。
-        id 1-6 は lerobot の SO-101 の割り当てと同じ。
+        PID の綴りは v0.2.2 に合わせて **わざと "cofficient"**（e 抜け）にしてある。
+        正しい綴りに直すと v0.2.2 は読まず、PID が一切設定されない。
+        driver を main 系へ上げるときは同時に直すこと。
       -->
-      <joint name="${prefix}shoulder_pan_joint">
-        <param name="id">1</param>
-        <command_interface name="position" />
-        <state_interface name="position" />
-        <state_interface name="velocity" />
-      </joint>
-      <joint name="${prefix}shoulder_lift_joint">
-        <param name="id">2</param>
-        <command_interface name="position" />
-        <state_interface name="position" />
-        <state_interface name="velocity" />
-      </joint>
-      <joint name="${prefix}elbow_flex_joint">
-        <param name="id">3</param>
-        <command_interface name="position" />
-        <state_interface name="position" />
-        <state_interface name="velocity" />
-      </joint>
-      <joint name="${prefix}wrist_flex_joint">
-        <param name="id">4</param>
-        <command_interface name="position" />
-        <state_interface name="position" />
-        <state_interface name="velocity" />
-      </joint>
-      <joint name="${prefix}wrist_roll_joint">
-        <param name="id">5</param>
-        <command_interface name="position" />
-        <state_interface name="position" />
-        <state_interface name="velocity" />
-      </joint>
-      <joint name="${prefix}gripper_joint">
-        <param name="id">6</param>
-        <command_interface name="position" />
-        <state_interface name="position" />
-        <state_interface name="velocity" />
-      </joint>
+      <xacro:macro name="sts_joint" params="name id offset p:=16 i:=0 d:=32">
+        <joint name="${prefix}${name}">
+          <param name="id">${id}</param>
+          <param name="offset">${offset}</param>
+          <param name="p_cofficient">${p}</param>
+          <param name="i_cofficient">${i}</param>
+          <param name="d_cofficient">${d}</param>
+          <command_interface name="position"/>
+          <state_interface name="position"/>
+          <state_interface name="velocity"/>
+        </joint>
+      </xacro:macro>
+      <xacro:sts_joint name="shoulder_pan_joint"  id="1" offset="${so101_offset_shoulder_pan}"/>
+      <xacro:sts_joint name="shoulder_lift_joint" id="2" offset="${so101_offset_shoulder_lift}"/>
+      <xacro:sts_joint name="elbow_flex_joint"    id="3" offset="${so101_offset_elbow_flex}"/>
+      <xacro:sts_joint name="wrist_flex_joint"    id="4" offset="${so101_offset_wrist_flex}"/>
+      <xacro:sts_joint name="wrist_roll_joint"    id="5" offset="${so101_offset_wrist_roll}"/>
+      <xacro:sts_joint name="gripper_joint"       id="6" offset="${so101_offset_gripper}"/>
     </ros2_control>
   </xacro:macro>

Commit message: fix: P ゲインを工場出荷値 32 へ戻し、再ビルド不要の開発オーバーレイを追加
■ 対話型で保持力が弱い件
lerobot が so_follower.configure() で P_Coefficient を 16 に下げている
(STS3215 の既定は 32。コメントは "to avoid shakiness")。それを xacro に
そのまま写していた。

位置制御のトルクは概ね P x 位置偏差。send_goal は時間軸のある軌道なので
指令が実位置を先行して偏差が持続するが、対話操作は指令が実位置に張り付いて
偏差がほぼゼロになる。「対話型でだけ弱い」の説明になる。

so101_p_gain を 32 (工場出荷値) へ戻した。PID は xacro 冒頭のプロパティに
切り出したので調整しやすい。振動したら 24 -> 20 -> 16 と下げる。

so101_probe に set_pid を追加。ROSを止めた状態でEEPROMへ直接書けるので、
値を探す実験が速い (次回起動時に URDF の値で上書きされる旨も表示する)。

■ 設定変更のたびに docker compose build が要る問題
イメージは --symlink-install でビルドしており、install 空間は symlink。
連鎖は install -> build -> src で、最終的に /ros2_ws/src を読んでいる。
つまりソースをマウントすれば再ビルド不要だった。この利点を使っていなかった。

compose.dev.yaml を追加:
    docker compose -f compose.yaml -f compose.dev.yaml up
config/control/launch/Python の編集が再起動だけで反映される。
新規ファイル追加や setup.py 変更は従来どおり再ビルドが必要。

Mac で検証: ホスト側の offset を 2048 -> 3999 に変えてオーバーレイ有りで
起動すると 3999 が反映され、オーバーレイ無しでは 2048 のままだった。

本番では使わない旨 (再現性が失われる) も明記した。

Co-Authored-By: Claude <noreply@anthropic.com>

File: ros2_ws/src/so101_bringup/control/so101_follower.ros2_control.xacro (robot description, xacro)
@@ -29,4 +29,21 @@
   <!-- 機体ごとの offset（URDF ゼロにおける Present tick）-->
   <xacro:include filename="$(find so101_bringup)/config/so101_offsets.xacro"/>
+  <!--
+    ★ サーボの PID。ここが「保持力の強さ」を決める調整ノブ。
+    位置制御のトルクは概ね `P × 位置偏差` なので、P が小さいと
+    **偏差が小さい場面で力が出ない**。
+      send_goal … 時間軸のある軌道で指令が実位置を先行 → 偏差が持続 → 力が出る
+      対話操作  … 指令が実位置に張り付く → 偏差ほぼゼロ → 力が出ない
+    「対話型でだけ弱い」のはこれが原因。
+    STS3215 の工場出荷値は P=32。lerobot は so_follower.configure() で
+    振動(shakiness)回避のため 16 へ下げているが、そのぶん保持力が落ちる。
+    ここでは **工場出荷値の 32 に戻している**。
+    振動する場合は 24 → 20 → 16 と下げること。
+    実機で素早く試すには so101_probe の set_pid オプションが使える
+    (docker/so101_ros2/README.md 参照)。値が決まったらここへ書き戻す。
+  -->
+  <xacro:property name="so101_p_gain" value="32"/>
+  <xacro:property name="so101_i_gain" value="0"/>
+  <xacro:property name="so101_d_gain" value="32"/>
   <xacro:macro
     name="ros2_control"
@@ -49,5 +66,7 @@
         driver を main 系へ上げるときは同時に直すこと。
       -->
-      <xacro:macro name="sts_joint" params="name id offset p:=16 i:=0 d:=32">
+      <xacro:macro name="sts_joint"
+                   params="name id offset
+                           p:=${so101_p_gain} i:=${so101_i_gain} d:=${so101_d_gain}">
         <joint name="${prefix}${name}">
           <param name="id">${id}</param>
