Commit message: fix: wrist_roll の offset を実測値 2116 に確定
実機で測定した値の報告を受けて反映。lerobot がフルターン扱いで可動域を
記録しないため計算できず、暫定で 2048 (無補正) を置いていた関節。

併せて、対話型で力が弱い件について実機の --torque 出力で仮説を確認した。

  全関節が P=16 (STS3215 の工場出荷値 32 の半分。lerobot が振動回避で下げた値)
  id 1-5 はトルク上限が満載 (MaxTorque=TorqueLim=1000) で絞られていない
  弱いのは全関節でグリッパ限定ではない -> MaxTorque=500 は主因ではない
  操作は rqt_joint_trajectory_controller のスライダ = 偏差が小さい場面

位置制御のトルクは概ね P x 位置偏差。スライダ操作は指令が実位置に張り付いて
偏差がほぼゼロになるため、P が小さいと力が出ない。P=32 への変更が正しい対処。

Co-Authored-By: Claude <noreply@anthropic.com>

File: ros2_ws/src/so101_bringup/config/so101_offsets.xacro (robot description, xacro)
@@ -17,8 +17,8 @@
     elbow_flex       670..3051     1916      −132
     wrist_flex      1014..3350     2182      +134
-    wrist_roll         0..4095     2048        +0    ★暫定
+    wrist_roll         0..4095     2116       +68    実機で実測
     gripper         1961..3399     1961       −87    ★要確認
   ★ wrist_roll: lerobot がフルターン扱いで可動域を記録しないため計算できない。
-    2048（無補正）を暫定で置いている。RViz と実物を見比べて手で詰めること。
+    2026‑08‑02 に実機で実測して 2116 に確定した（暫定値 2048 から +68）。
   ★ gripper: 「閉」が range_min(1961) 側であることを未確認。
     閉じ切って so101_probe の Present を読み、range_max(3399) 側だったら
@@ -32,5 +32,5 @@
   <xacro:property name="so101_offset_elbow_flex"    value="1916"/>
   <xacro:property name="so101_offset_wrist_flex"    value="2182"/>
-  <xacro:property name="so101_offset_wrist_roll"    value="2048"/>
+  <xacro:property name="so101_offset_wrist_roll"    value="2116"/>
   <xacro:property name="so101_offset_gripper"       value="1961"/>
 </robot>
