Commit message: feat: 前方 120° スキャンフィルターを追加し、後方車輪の幻障害物を排除
後方車輪(180°)やボディが /scan に映ると、SLAM の地図とコストマップに
幻の壁が焼き付く問題に対処した。

変更内容:
- scan_filter.py を追加: /scan を右車輪(-60°)〜左車輪(+60°)の前方 120°
  アークにフィルタリングして /scan_filtered として配信する ROS 2 ノード
- nav.launch.py / nav_with_map.launch.py に scan_angular_filter ノードを追加
- slam_toolbox.yaml の scan_topic を /scan_filtered へ変更
- nav2.yaml の local_costmap / global_costmap / collision_monitor の
  スキャントピックを /scan_filtered へ変更
- URDF の laser_link 位置を実測値 (0.10 0 0.03) に更新

Co-Authored-By: Claude Sonnet 4.6 <noreply@anthropic.com>

File: ros2_ws/src/lekiwi_description/urdf/lekiwi_base.macro.xacro (robot description, xacro)
@@ -47,5 +47,5 @@
     <xacro:property name="cad_yaw" value="${-pi/2}"/>
     <!-- ★ TBD: 実測待ち。RViz でマゼンタ表示されるので未確定と分かる ★ -->
-    <xacro:property name="laser_xyz_TBD" value="0 0 0.09"/>
+    <xacro:property name="laser_xyz_TBD" value="0.10 0 0.03"/>
     <xacro:property name="laser_rpy_TBD" value="0 0 0"/>
     <!-- カメラマウントは CAD 由来 (CAD (0.02, 0.1, 0) → base_link (0.1, -0.02, 0))。
