Commit message: Harden SO101 reach lifecycle and set LiDAR yaw

File: ros2_ws/src/lekiwi_description/urdf/lekiwi_base.macro.xacro (robot description, xacro)
@@ -46,7 +46,7 @@
     <!-- CAD 座標系 → base_link の回転。メッシュを使う場合に必要 -->
     <xacro:property name="cad_yaw" value="${-pi/2}"/>
-    <!-- ★ TBD: 実測待ち。RViz でマゼンタ表示されるので未確定と分かる ★ -->
-    <xacro:property name="laser_xyz_TBD" value="0.10 0 0.03"/>
-    <xacro:property name="laser_rpy_TBD" value="0 0 0"/>
+    <!-- LiDAR回転中心: x=100 mm, y=0 mm, z=30 mm。yaw=-7 deg指定 -->
+    <xacro:property name="laser_xyz" value="0.10 0 0.03"/>
+    <xacro:property name="laser_rpy" value="0 0 -0.1221730476"/>
     <!-- カメラマウントは CAD 由来 (CAD (0.02, 0.1, 0) → base_link (0.1, -0.02, 0))。
          光学フレームのオフセットは未実測。 -->
@@ -184,5 +184,5 @@
     <!-- ================= センサ取付フレーム (未実測) ================= -->
     <!--
-      ★ laser_link の位置は未実測。RPLIDAR A1 を載せたら実測して差し替えること。
+      ★ laser_link の位置はRPLIDAR A1実機で実測済み。
         フレーム名の整合は rplidar_bringup 側で取ってある。sllidar_ros2 の
         既定の frame_id は "laser" だが、a1_points.launch.py が
@@ -193,5 +193,5 @@
     -->
     <joint name="${prefix}laser_joint" type="fixed">
-      <origin xyz="${laser_xyz_TBD}" rpy="${laser_rpy_TBD}"/>
+      <origin xyz="${laser_xyz}" rpy="${laser_rpy}"/>
       <parent link="${prefix}base_link"/>
       <child link="${prefix}laser_link"/>
@@ -225,13 +225,12 @@
     </link>
     <!--
-      アーム取付位置。CAD (0.04, 0.08, 0.057) → base_link (0.08, -0.04, 0.057)。
+      アーム取付位置。実測値 base_link (0.08, 0.00, 0.057)。
       SO-101 を載せる構成は lekiwi_so101_bringup を参照 (このマクロ単体では何も生えない)。
-      ★ この値は CAD 由来で実測していない。特にブラケットの向き (yaw) は未確認。
-        laser_xyz_TBD と同じく実測待ちなので、確定するまで数 cm の誤差を前提にすること。
+      ★ x/y/z とブラケットの向き (yaw) は実機で実測した値。
       ★ 電源系の注意: アームは 7.4V、ホイールは 12V。同一バスへ繋いではいけない。
         アームを載せても給電とシリアルバスは別系統のまま保つこと。
     -->
     <joint name="${prefix}arm_mount_joint" type="fixed">
-      <origin xyz="0.08 -0.04 0.057" rpy="0 0 0"/>
+      <origin xyz="0.08 0.00 0.057" rpy="0 0 0"/>
       <parent link="${prefix}base_link"/>
       <child link="${prefix}arm_mount_link"/>

File: ros2_ws/src/lekiwi_so101_bringup/urdf/lekiwi_so101.urdf.xacro (robot description, xacro)
@@ -29,8 +29,8 @@
   <xacro:arg name="ros2_control_file"
              default="$(find so101_bringup)/control/so101_follower.ros2_control.xacro"/>
-  <!-- ★ TBD: 実測待ち。arm_mount_link から見たアーム基部の姿勢。
-       arm_mount_link 自体 (base_link から 0.08, -0.04, 0.057) も CAD 由来で未実測。
-       特に yaw はブラケットの向き次第で 90 度単位で変わりうる。
-       docs/agent/request.md の手順 0 と 3 で確定させること。
+  <!-- ★ arm_mount_link の位置は実測済み: base_link から (0.08, 0.00, 0.057)。
+       以下は arm_mount_link から見たアーム基部の姿勢。
+       取付姿勢 (roll/pitch/yaw) は実測値を使用する。
+       docs/agent/request.md の手順 3 でTFを照合すること。
        xacro のマクロ引数はベクトルを展開できないのでスカラ 6 個で渡す。 -->
   <xacro:arg name="arm_mount_x" default="0.0"/>

Commit message: Update measured LeKiwi plate heights

File: ros2_ws/src/lekiwi_description/urdf/lekiwi_base.macro.xacro (robot description, xacro)
@@ -31,17 +31,14 @@
                        base_radius:=0.125">
     <!-- ================= 寸法 (CAD 由来) ================= -->
-    <!-- 車軸の高さ。base_link 原点 (= CAD 原点) からの実測値 -->
-    <xacro:property name="axle_z" value="0.01786"/>
-    <!-- 接地面から base_link までの高さ。
-         CAD 実測では 0.032924 m (このとき車輪半径 0.050784 m)。
-         wheel_radius から導出しておけば、公称 0.05 を使っても車輪が
-         きっちり接地する。 -->
-    <xacro:property name="base_link_z" value="${wheel_radius - axle_z}"/>
+    <!-- 下段プレート上面 (= base_link 原点) の地面からの実測値。 -->
+    <xacro:property name="base_link_z" value="0.040"/>
+    <!-- 車軸の高さ。車輪が地面に接するよう、車輪半径から導出する。 -->
+    <xacro:property name="axle_z" value="${wheel_radius - base_link_z}"/>
     <xacro:property name="wheel_width" value="0.026"/>  <!-- 仮値: 見た目のみ -->
     <!-- ベースプレート: CAD bbox [-107.9,-105,-7]..[107.9,107.9,0] mm -->
     <xacro:property name="plate_size" value="0.216"/>
     <xacro:property name="plate_thickness" value="0.007"/>
-    <!-- 第2プレート: base_link から +0.05 m -->
-    <xacro:property name="plate2_z" value="0.05"/>
+    <!-- 第2プレート: 上面間の実測値 92 - 40 = 52 mm -->
+    <xacro:property name="plate2_z" value="0.052"/>
     <!-- CAD 座標系 → base_link の回転。メッシュを使う場合に必要 -->
     <xacro:property name="cad_yaw" value="${-pi/2}"/>
