Commit message: feat: RealSense を手首カメラとして載せ、点群を map 上に置く
feat/lekiwi-so101-reach から分岐。アームの arm_gripper_link に
RealSense D435i を載せ、点群が map 上の正しい位置に出るようにした。

■ ★ 手首カメラは外部キャリブレーションが要らない
別ブランチ feat/env-camera の「環境固定カメラ」は map 原点が物理的な印でない
ため、マーカーや ICP で map -> camera を推定する必要があった。手首カメラは
URDF のリンクに剛体固定されるので、

  map -> ... -> arm_gripper_link -> wrist_camera_mount_link
             -> wrist_camera_link -> wrist_camera_depth_optical_frame

がすべて URDF と /joint_states から出る。**env-camera の env_camera_calib.py /
gravity.py / icp2d.py (約 700 行) は丸ごと不要**で、このブランチでは
**新規ノードがゼロ**。

■ URDF での繋ぎ方 (ここが要点)
wrist_camera_link を**この URDF 側で宣言し、mount の子にする**。
realsense2_camera は <camera_name>_link を自分のサブツリーの根として
<name>_link -> <name>_depth_frame などを /tf_static へ出すが、
**<name>_link を子にする TF は出さない**ので、親をこちらが与えても
二重定義にならない。lekiwi_description の laser_link と同じパターン。
実際に結合 URDF を展開し、wrist_camera_link を子とする joint が
ちょうど 1 個であることを確認した。

★ カメラのフレームにアームの接頭辞は付けない。アーム側は上流マクロが arm_ を
付けるが、カメラのフレーム名は realsense の camera_name パラメータから作られる。

★ 上流の so_arm101_macro.xacro は vendoring 禁止対象なので触らず、結合 xacro
側で ${prefix}gripper_link に生やした。

■ d435i.launch.py を feat/env-camera から移植
手首でも同じ修正が要る。特に **camera_name を parameters= に渡さないと
フレーム名が camera_link から動かない**バグ (name=/namespace= はトピックにしか
効かない)。点群の有効化、pointcloud_qos: SENSOR_DATA、fps 引数が実際には
効いていなかった件、hole_filling を無効にする判断も含む。
enable_imu は既定 false のまま残した (手首では不要だが、ブランチ間の
無用な分岐を避けるため)。

■ Mac のモックで確認したこと
- 結合 URDF が単一ツリーのまま、リンク名の重複なし
- arm_gripper_link -> wrist_camera_mount_link -> wrist_camera_link
- **★ 腕を動かすとカメラ TF が追従する**（固定カメラとの決定的な違い）:
  map -> wrist_camera_link が (0.230,-0.115,0.210) -> (0.312,0.199,0.388)。
  arm_gripper_link と完全に一致する（取付オフセットが 0 なので当然）
- **★ 光学フレームの軸の検算**: 光学系 (x右 y下 z前) の +z 0.3m 前方が、
  camera_link 系の +x 0.3m 前方と同一点になることを tf2 で確認 (1e-6 以内)。
  模擬光学フレーム (mock_wrist_camera_optical) を足して Mac で検証できるようにした
- make check に map -> wrist_camera_depth_optical_frame を追加
- pytest 28 passed / 9 skipped

■ 実機に持っていく前に見るべきリスク (README と実機手順に記載)
- **★ 積載重量**: D435i 約 72g + マウント + ケーブル。アームは約 750g で
  全関節 P=16 の保持力問題が未解決。手首の先端に足すのは悪化側に効く。
  無通電で取り付けて手を離し、姿勢を保てるかを最初に見るべき
- USB ケーブルが抵抗トルクと可動域制限になる
- joint_limit_overrides は空のまま。干渉体が増える
- stow_positions が無効になりうる
- 視野に arm_jaw_link が入る
- **D435i の最短測距 (約 0.1〜0.2m)**。手首カメラは対象に近づくので、
  リーチ目標の距離では測距範囲を下回る可能性がある。用途の成否に関わる

未検証: 実機すべて。パラメータ名 (pointcloud.stream_filter)、帯域、
取付姿勢の実測、ケーブルの可動域制限。

File: ros2_ws/src/lekiwi_so101_bringup/urdf/lekiwi_so101.urdf.xacro (robot description, xacro)
@@ -40,4 +40,18 @@
   <xacro:arg name="arm_mount_pitch" default="0.0"/>
   <xacro:arg name="arm_mount_yaw" default="0.0"/>
+  <!-- ★ 手首カメラ (RealSense D435i)。
+       取り付けは arm_gripper_link。wrist_roll と一緒に回るので、
+       リーチのソルバが wrist_roll を凍結する以上ロール角は一定になる。
+       ★ 取付姿勢は未実測。arm_mount / laser と同じ TBD 流儀で、
+         確定するまでマゼンタのマーカーで見えるようにしてある。 -->
+  <xacro:arg name="wrist_camera" default="true"/>
+  <xacro:arg name="wrist_camera_name" default="wrist_camera"/>
+  <xacro:arg name="wrist_camera_parent" default="gripper_link"/>
+  <xacro:arg name="wrist_camera_x" default="0.0"/>
+  <xacro:arg name="wrist_camera_y" default="0.0"/>
+  <xacro:arg name="wrist_camera_z" default="0.0"/>
+  <xacro:arg name="wrist_camera_roll" default="0.0"/>
+  <xacro:arg name="wrist_camera_pitch" default="0.0"/>
+  <xacro:arg name="wrist_camera_yaw" default="0.0"/>
   <xacro:include filename="$(find lekiwi_description)/urdf/lekiwi_base.macro.xacro"/>
   <xacro:lekiwi_base prefix=""
@@ -55,4 +69,53 @@
                    pitch="$(arg arm_mount_pitch)"
                    yaw="$(arg arm_mount_yaw)"/>
+  <!-- ================= 手首カメラ ================= -->
+  <!--
+    ★ ここが「点群を map 上に置く」ための全て。外部キャリブレーションは要らない。
+      map -> ... -> ${prefix}gripper_link
+                 -> wrist_camera_mount_link      (この URDF)
+                 -> wrist_camera_link            (この URDF)
+                 -> wrist_camera_depth_optical_frame  (realsense2_camera が /tf_static へ)
+    ★ wrist_camera_link を**この URDF 側で宣言し、mount の子にする**のが要点。
+      realsense2_camera は <camera_name>_link を自分のサブツリーの根として
+      <name>_link -> <name>_depth_frame などを出すが、<name>_link を**子にする
+      TF は出さない**。したがって親をこちらが与えても二重定義にならない。
+      lekiwi_description の laser_link と同じパターン。
+    ★ カメラのフレームにアームの接頭辞 (${prefix}) は付けない。
+      アーム側のリンク名は上流マクロが prefix を付けるが、カメラのフレーム名は
+      realsense2_camera の camera_name パラメータから作られるため。
+      launch の camera_name と wrist_camera_name を必ず一致させること。
+  -->
+  <xacro:if value="$(arg wrist_camera)">
+    <joint name="$(arg wrist_camera_name)_mount_joint" type="fixed">
+      <origin xyz="$(arg wrist_camera_x) $(arg wrist_camera_y) $(arg wrist_camera_z)"
+              rpy="$(arg wrist_camera_roll) $(arg wrist_camera_pitch) $(arg wrist_camera_yaw)"/>
+      <parent link="$(arg prefix)$(arg wrist_camera_parent)"/>
+      <child link="$(arg wrist_camera_name)_mount_link"/>
+    </joint>
+    <!-- TBD マーカー。RViz で取付位置が未確定だと分かるようにする。 -->
+    <link name="$(arg wrist_camera_name)_mount_link">
+      <visual>
+        <geometry>
+          <box size="0.02 0.02 0.004"/>
+        </geometry>
+        <material name="lekiwi_tbd"/>
+      </visual>
+    </link>
+    <!-- D435i の筐体 (90 x 25 x 25 mm)。camera_link は筐体の中心ではなく
+         左赤外イメージャ基準だが、見た目の目安として置く。 -->
+    <joint name="$(arg wrist_camera_name)_link_joint" type="fixed">
+      <origin xyz="0 0 0" rpy="0 0 0"/>
+      <parent link="$(arg wrist_camera_name)_mount_link"/>
+      <child link="$(arg wrist_camera_name)_link"/>
+    </joint>
+    <link name="$(arg wrist_camera_name)_link">
+      <visual>
+        <geometry>
+          <box size="0.025 0.090 0.025"/>
+        </geometry>
+        <material name="lekiwi_tbd"/>
+      </visual>
+    </link>
+  </xacro:if>
   <xacro:include filename="$(arg ros2_control_file)"/>
   <xacro:ros2_control prefix="$(arg prefix)"

Commit message: fix: wrist camera pitchを65度に更新

File: ros2_ws/src/lekiwi_so101_bringup/urdf/lekiwi_so101.urdf.xacro (robot description, xacro)
@@ -43,16 +43,7 @@
        取り付けは arm_gripper_link。wrist_roll と一緒に回るので、
        リーチのソルバが wrist_roll を凍結する以上ロール角は一定になる。
-       ★★ 既定値は **実測値ではない**。公式 STL から幾何計算した参考値であり、
-          しかも **D405 + Wrist_Roll_D405_Holder を前提とした値**。
-          手元の D435i には SO-101 用の公式マウントが存在しないため、
-          この値がそのまま正しくなる構成は現時点では無い。
-          「0 よりマシな初期値」以上の意味を持たせないこと。
-          導出の根拠と再計算手順は docs/wrist_camera.md の
-          「幾何計算による参考値」節。要点だけ:
-            - SO101/assets の asset と公式 STL は同一座標系 (bbox 完全一致)
-            - D405 の M3 取付穴は背面 (Ø2.48 x2, 20.00mm)。光軸は取付面に垂直
-            - 誤差 ±2mm / ±2 度。roll は ±180 度の曖昧さが残る
-          W-5 で実測値が出たら .env で上書きし、確定したらここも差し替える。
-       ★ 未実測であることに変わりはないので、TBD マーカー (マゼンタ) は残す。 -->
+       ★ wrist_camera_* は固定台ではなく、webcam の基準位置・姿勢を表す。
+         webcam 用固定台から見たカメラの位置・向きを先に反映し、
+         D435i のレンズ中心との差だけを後段で補正する。 -->
   <xacro:arg name="wrist_camera" default="true"/>
   <xacro:arg name="wrist_camera_name" default="wrist_camera"/>
@@ -62,5 +53,5 @@
   <xacro:arg name="wrist_camera_z" default="-0.02074"/>
   <xacro:arg name="wrist_camera_roll" default="3.14159"/>
-  <xacro:arg name="wrist_camera_pitch" default="1.04718"/>
+  <xacro:arg name="wrist_camera_pitch" default="1.13445"/>
   <xacro:arg name="wrist_camera_yaw" default="1.57080"/>
   <xacro:include filename="$(find lekiwi_description)/urdf/lekiwi_base.macro.xacro"/>
@@ -98,10 +89,9 @@
   <xacro:if value="$(arg wrist_camera)">
     <joint name="$(arg wrist_camera_name)_mount_joint" type="fixed">
-      <origin xyz="$(arg wrist_camera_x) $(arg wrist_camera_y) $(arg wrist_camera_z)"
-              rpy="$(arg wrist_camera_roll) $(arg wrist_camera_pitch) $(arg wrist_camera_yaw)"/>
+      <origin xyz="0 0 0" rpy="0 0 0"/>
       <parent link="$(arg prefix)$(arg wrist_camera_parent)"/>
       <child link="$(arg wrist_camera_name)_mount_link"/>
     </joint>
-    <!-- TBD マーカー。RViz で取付位置が未確定だと分かるようにする。 -->
+    <!-- gripper_link 直下の中継フレーム。位置の基準はここでは持たない。 -->
     <link name="$(arg wrist_camera_name)_mount_link">
       <visual>
@@ -112,8 +102,9 @@
       </visual>
     </link>
-    <!-- D435i の筐体 (90 x 25 x 25 mm)。camera_link は筐体の中心ではなく
-         左赤外イメージャ基準だが、見た目の目安として置く。 -->
+    <!-- webcam 基準位置に置くカメラフレーム。
+         D435i の筐体 (90 x 25 x 25 mm) は見た目の目安として置く。 -->
     <joint name="$(arg wrist_camera_name)_link_joint" type="fixed">
-      <origin xyz="0 0 0" rpy="0 0 0"/>
+      <origin xyz="$(arg wrist_camera_x) $(arg wrist_camera_y) $(arg wrist_camera_z)"
+              rpy="$(arg wrist_camera_roll) $(arg wrist_camera_pitch) $(arg wrist_camera_yaw)"/>
       <parent link="$(arg wrist_camera_name)_mount_link"/>
       <child link="$(arg wrist_camera_name)_link"/>
